File: Schematic_Scraps/Display.kicad_sch (KiCad schematic)
At the start: 6 parts, among them IC17 K155ЛН2/7405, IC18 K155ЛН2/7405, IC19 K155ЛН2/7405, IC20 K155ЛН2/7405, J3 Conn_02x13_Counter_Clockwise, U15 КР580ВВ55А/8255

Commit message: Further reverse engineering progress
Parts:
- J3: value Conn_02x13_Counter_Clockwise -> To 7-seg. Display
- renumbered IC17 to U17, IC18 to U18, IC19 to U19
Connections:
- net GND: now also J3.10 (Pin_10); no longer J3.17 (Pin_17)
- net RESET: now reaches U15.35 (RESET)
- net ~{PPI2_PB2}: now reaches J3.26 (Pin_26)
- net ~{PPI2_PB2}: now also U18.8
- net PA0 renamed PPI2_PA0
- net PA1 renamed PPI2_PA1
- net PA2 renamed PPI2_PA2
- net PA3 renamed PPI2_PA3
- net PA4 renamed PPI2_PA4
- net PA5 renamed PPI2_PA5
- net PA6 renamed PPI2_PA6
- net PA7 renamed PPI2_PA7
- net PB0 renamed PPI2_PB0
- net PB1 renamed PPI2_PB1
- net PB2 renamed PPI2_PB2
- net PB3 renamed PPI2_PB3
- net PB4 renamed PPI2_PB4
- net PB5 renamed PPI2_PB5
- net PB6 renamed PPI2_PB6
- net PB7 renamed PPI2_PB7
- net PC0 renamed PPI2_PC0
- net PC1 renamed PPI2_PC1
- net PC2 renamed PPI2_PC2
- net PC3 renamed PPI2_PC3
- net PC4 renamed PPI2_PC4
- net PC5 renamed PPI2_PC5
- net PC6 renamed PPI2_PC6
- net PC7 renamed PPI2_PC7
- net ~{PA0} renamed ~{PPI2_PA0}
- net ~{PPI2_PA0}: now also J3.9 (Pin_9); no longer J3.18 (Pin_18)
- net ~{PA1} renamed ~{PPI2_PA1}
- net ~{PPI2_PA1}: now also J3.16 (Pin_16); no longer J3.11 (Pin_11)
- net ~{PA2} renamed ~{PPI2_PA2}
- net ~{PPI2_PA2}: now also J3.15 (Pin_15); no longer J3.12 (Pin_12)
- net ~{PA3} renamed ~{PPI2_PA3}
- net ~{PPI2_PA3}: now also J3.14 (Pin_14); no longer J3.13 (Pin_13)
- net ~{PA4} renamed ~{PPI2_PA4}
- net ~{PPI2_PA4}: now also J3.13 (Pin_13); no longer J3.14 (Pin_14)
- net ~{PA5} renamed ~{PPI2_PA5}
- net ~{PPI2_PA5}: now also J3.12 (Pin_12); no longer J3.15 (Pin_15)
- net ~{PA6} renamed ~{PPI2_PA6}
- net ~{PPI2_PA6}: now also J3.11 (Pin_11); no longer J3.16 (Pin_16)
- net ~{PA7} renamed ~{PPI2_PA7}
- net ~{PPI2_PA7}: now also J3.17 (Pin_17); no longer J3.10 (Pin_10)
- net ~{PB0} renamed ~{PPI2_PB0}
- net ~{PPI2_PB0}: now also J3.24 (Pin_24); no longer J3.3 (Pin_3)
- net ~{PB1} renamed ~{PPI2_PB1}
- net ~{PPI2_PB1}: now also J3.25 (Pin_25); no longer J3.2 (Pin_2)
- net ~{PB2} renamed SPEAKER
- net SPEAKER: no longer U18.8
- net ~{PB3} renamed ~{PPI2_PB3}
- net ~{PPI2_PB3}: now also J3.2 (Pin_2); no longer J3.25 (Pin_25)
- net ~{PB4} renamed ~{PPI2_PB4}
- net ~{PPI2_PB4}: now also J3.3 (Pin_3); no longer J3.24 (Pin_24)
- net ~{PB5} renamed ~{PPI2_PB5}
- net ~{PPI2_PB5}: now also J3.23 (Pin_23); no longer J3.4 (Pin_4)
- net ~{PB6} renamed ~{PPI2_PB6}
- net ~{PPI2_PB6}: now also J3.4 (Pin_4); no longer J3.23 (Pin_23)
- net ~{PB7} renamed ~{PPI2_PB7}
- net ~{PPI2_PB7}: now also J3.5 (Pin_5); no longer J3.22 (Pin_22)
- net ~{PC0} renamed ~{PPI2_PC0}
- net ~{PPI2_PC0}: now also J3.20 (Pin_20); no longer J3.7 (Pin_7)
- net ~{PC1} renamed ~{PPI2_PC1}
- net ~{PPI2_PC1}: now also J3.6 (Pin_6); no longer J3.21 (Pin_21)
- net ~{PC2} renamed ~{PPI2_PC2}
- net ~{PPI2_PC2}: now also J3.21 (Pin_21); no longer J3.6 (Pin_6)
- net ~{PC3} renamed ~{PPI2_PC3}
- net ~{PPI2_PC3}: now also J3.22 (Pin_22); no longer J3.5 (Pin_5)
- net ~{PC4} renamed ~{PPI2_PC4}
- net ~{PPI2_PC4}: now also J3.7 (Pin_7); no longer J3.20 (Pin_20)
- net ~{PC5} renamed ~{PPI2_PC5}
- net ~{PPI2_PC5}: now also J3.19 (Pin_19); no longer J3.8 (Pin_8)
- net ~{PC6} renamed ~{PPI2_PC6}
- net ~{PPI2_PC6}: now also J3.18 (Pin_18); no longer J3.9 (Pin_9)
- net ~{PC7} renamed ~{PPI2_PC7}
- net ~{PPI2_PC7}: now also J3.8 (Pin_8); no longer J3.19 (Pin_19)
Other:
- company: (none) -> Brett Hallen
- title: (none) -> Rhythm Keyboard (Ритм Клав)
- moved on the sheet: IC20A, IC20B, IC20C, IC20D, IC20E, IC20F, J3, U17B, U17C, U17D, U17E, U18A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
