File: Schematic_Scraps/Interface.kicad_sch (KiCad schematic)
At the start: 9 parts, among them J1 Conn_01x09, J2 Cassette, U1 АОТ101АС (ILD74), U2 К555ТЛ2 (74LS14), U3 КР580ВВ51А (8251)

Commit message: Analysis progress
Connections:
- net D2: now reaches U3.1 (D_{2})
- net D3: now reaches U3.2 (D_{3})
- net D0: now reaches U3.27 (D_{0})
- net D1: now reaches U3.28 (D_{1})
- net D4: now reaches U3.5 (D_{4})
- net D5: now reaches U3.6 (D_{5})
- net D6: now reaches U3.7 (D_{6})
- net D7: now reaches U3.8 (D_{7})
- no-connect marks 0 -> 2
Changed lines of the file:
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@@
 	(generator_version "9.0")
 	(paper "A4")
-	(text_box "АОТ101АС = ILD74\nК555ТЛ2 = 74LS14\nКР580ГФ24 = Intel 8224"
-		(exclude_from_sim no)
-		(at 201.93 124.46 0)
-		(size 53.34 34.29)
-		(margins 0.9525 0.9525 0.9525 0.9525)
-		(stroke
-			(width 0)
-			(type solid)
-		)
-		(fill
-			(type none)
-		)
-		(effects
-			(font
-				(size 1.27 1.27)
-			)
-			(justify left top)
-		)
-	)
 	(junction
 		(at 157.48 67.31)
@@
 		(color 0 0 0 0)
 	)
+	(no_connect
+		(at 88.9 39.37)
+	)
+	(no_connect
+		(at 73.66 39.37)
+	)
 	(wire
 		(pts
@@
 	(wire
 		(pts
-			(xy 82.55 76.2) (xy 74.93 76.2)
+			(xy 71.12 76.2) (xy 82.55 76.2)
 		)
 		(stroke
@@
 	(wire
 		(pts
-			(xy 274.32 27.94) (xy 274.32 25.4)
-		)
-		(stroke
-			(width 0)
-			(type default)
-		)
-	)
-	(wire
-		(pts
-			(xy 74.93 76.2) (xy 74.93 60.96)
+			(xy 278.13 22.86) (xy 278.13 20.32)
+		)
+		(stroke
+			(width 0)
+			(type default)
+		)
+	)
+	(wire
+		(pts
+			(xy 71.12 76.2) (xy 71.12 60.96)
 		)
 		(stroke
@@
 	(wire
 		(pts
-			(xy 74.93 60.96) (xy 127 60.96)
+			(xy 71.12 60.96) (xy 127 60.96)
 		)
 		(stroke
@@
 	(wire
 		(pts
-			(xy 257.81 26.67) (xy 257.81 27.94)
+			(xy 278.13 30.48) (xy 278.13 31.75)
 		)
 		(stroke
@@
 	(wire
 		(pts
-			(xy 238.76 27.94) (xy 238.76 26.67)
+			(xy 278.13 40.64) (xy 278.13 39.37)
 		)
 		(stroke
@@
 	)
 	(label "-12V input"
-		(at 274.32 27.94 180)
+		(at 278.13 22.86 180)
 		(effects
 			(font
@@
 	)
 	(label "+5V input"
-		(at 238.76 27.94 180)
+		(at 278.13 40.64 180)
 		(effects
 			(font
@@
 	)
 	(label "RxD"
-		(at 82.55 76.2 180)
+		(at 76.2 76.2 180)
 		(effects
 			(font
@@
 	)
 	(label "+12V input"
-		(at 257.81 27.94 180)
+		(at 278.13 31.75 180)
 		(effects
 			(font
@@
 		)
 	)
+	(global_label "D3"
+		(shape input)
+		(at 82.55 73.66 180)
+		(fields_autoplaced yes)
+		(effects
+			(font
+				(size 1.27 1.27)
+			)
+			(justify right)
+		)
+		(property "Intersheetrefs" "${INTERSHEET_REFS}"
+			(at 77.0853 73.66 0)
+			(effects
+				(font
+					(size 1.27 1.27)
+				)
+				(justify right)
+				(hide yes)
+			)
+		)
+	)
+	(global_label "D1"
+		(shape input)
+		(at 107.95 71.12 0)
+		(fields_autoplaced yes)
+		(effects
+			(font
+				(size 1.27 1.27)
+			)
+			(justify left)
+		)
+		(property "Intersheetrefs" "${INTERSHEET_REFS}"
+			(at 113.4147 71.12 0)
+			(effects
+				(font
+					(size 1.27 1.27)
+				)
+				(justify left)
+				(hide yes)
+			)
+		)
+	)
 	(global_label "~{8251}"
 		(shape input)
@@
 		(property "Intersheetrefs" "${INTERSHEET_REFS}"
 			(at 74.7268 96.52 0)
+			(effects
+				(font
+					(size 1.27 1.27)
+				)
+				(justify right)
+				(hide yes)
+			)
+		)
+	)
+	(global_label "D6"
+		(shape input)
+		(at 82.55 86.36 180)
+		(fields_autoplaced yes)
+		(effects
+			(font
+				(size 1.27 1.27)
+			)
+			(justify right)
+		)
+		(property "Intersheetrefs" "${INTERSHEET_REFS}"
+			(at 77.0853 86.36 0)
+			(effects
+				(font
+					(size 1.27 1.27)
+				)
+				(justify right)
+				(hide yes)
+			)
+		)
+	)
+	(global_label "D5"
+		(shape input)
+		(at 82.55 83.82 180)
+		(fields_autoplaced yes)
+		(effects
+			(font
+				(size 1.27 1.27)
+			)
+			(justify right)
+		)
+		(property "Intersheetrefs" "${INTERSHEET_REFS}"
+			(at 77.0853 83.82 0)
+			(effects
+				(font
+					(size 1.27 1.27)
+				)
+				(justify right)
+				(hide yes)
+			)
+		)
+	)
+	(global_label "D4"
+		(shape input)
+		(at 82.55 81.28 180)
+		(fields_autoplaced yes)
+		(effects
+			(font
+				(size 1.27 1.27)
+			)
+			(justify right)
+		)
+		(property "Intersheetrefs" "${INTERSHEET_REFS}"
+			(at 77.0853 81.28 0)
+			(effects
+				(font
+					(size 1.27 1.27)
+				)
+				(justify right)
+				(hide yes)
+			)
+		)
+	)
+	(global_label "D0"
+		(shape input)
+		(at 107.95 73.66 0)
+		(fields_autoplaced yes)
+		(effects
+			(font
+				(size 1.27 1.27)
+			)
+			(justify left)
+		)
+		(property "Intersheetrefs" "${INTERSHEET_REFS}"
+			(at 113.4147 73.66 0)
+			(effects
+				(font
+					(size 1.27 1.27)
+				)
+				(justify left)
+				(hide yes)
+			)
+		)
+	)
+	(global_label "D7"
+		(shape input)
+		(at 82.55 88.9 180)
+		(fields_autoplaced yes)
+		(effects
+			(font
+				(size 1.27 1.27)
+			)
+			(justify right)
+		)
+		(property "Intersheetrefs" "${INTERSHEET_REFS}"
+			(at 77.0853 88.9 0)
+			(effects
+				(font
+					(size 1.27 1.27)
+				)
+				(justify right)
+				(hide yes)
+			)
+		)
+	)
+	(global_label "D2"
+		(shape input)
+		(at 82.55 71.12 180)
+		(fields_autoplaced yes)
+		(effects
+			(font
+				(size 1.27 1.27)
+			)
+			(justify right)
+		)
+		(property "Intersheetrefs" "${INTERSHEET_REFS}"
+			(at 77.0853 71.12 0)
 			(effects
 				(font
@@
 	(symbol
 		(lib_id "power:+5V")
-		(at 238.76 26.67 0)
+		(at 278.13 39.37 0)
 		(unit 1)
 		(exclude_from_sim no)
@@
 		(fields_autoplaced yes)
 		(property "Reference" "#PWR03"
-			(at 238.76 30.48 0)
+			(at 278.13 43.18 0)
 			(effects
 				(font
@@
 		)
 		(property "Value" "+5V"
-			(at 238.76 21.59 0)
+			(at 278.13 34.29 0)
 			(effects
 				(font
@@
 		)
 		(property "Footprint" ""
-			(at 238.76 26.67 0)
+			(at 278.13 39.37 0)
 			(effects
 				(font
@@
 		)
 		(property "Datasheet" ""
-			(at 238.76 26.67 0)
+			(at 278.13 39.37 0)
 			(effects
 				(font
@@
 		)
 		(property "Description" "Power symbol creates a global label with name \"+5V\""
-			(at 238.76 26.67 0)
+			(at 278.13 39.37 0)
 			(effects
 				(font
@@
 	(symbol
 		(lib_id "power:+12V")
-		(at 257.81 26.67 0)
+		(at 278.13 30.48 0)
 		(unit 1)
 		(exclude_from_sim no)
@@
 		(fields_autoplaced yes)
 		(property "Reference" "#PWR08"
-			(at 257.81 30.48 0)
+			(at 278.13 34.29 0)
 			(effects
 				(font
@@
 		)
 		(property "Value" "+12V"
-			(at 257.81 21.59 0)
+			(at 278.13 25.4 0)
 			(effects
 				(font
@@
 		)
 		(property "Footprint" ""
-			(at 257.81 26.67 0)
+			(at 278.13 30.48 0)
 			(effects
 				(font
@@
 		)
 		(property "Datasheet" ""
-			(at 257.81 26.67 0)
+			(at 278.13 30.48 0)
 			(effects
 				(font
@@
 		)
 		(property "Description" "Power symbol creates a global label with name \"+12V\""
-			(at 257.81 26.67 0)
+			(at 278.13 30.48 0)
 			(effects
 				(font
@@
 	(symbol
 		(lib_id "power:-12V")
-		(at 274.32 25.4 0)
+		(at 278.13 20.32 0)
 		(unit 1)
 		(exclude_from_sim no)
@@
 		(fields_autoplaced yes)
 		(property "Reference" "#PWR09"
-			(at 274.32 29.21 0)
+			(at 278.13 24.13 0)
 			(effects
 				(font
@@
 		)
 		(property "Value" "-12V"
-			(at 274.32 20.32 0)
+			(at 278.13 15.24 0)
 			(effects
 				(font
@@
 		)
 		(property "Footprint" ""
-			(at 274.32 25.4 0)
+			(at 278.13 20.32 0)
 			(effects
 				(font
@@
 		)
 		(property "Datasheet" ""
-			(at 274.32 25.4 0)
+			(at 278.13 20.32 0)
 			(effects
 				(font
@@
 		)
 		(property "Description" "Power symbol creates a global label with name \"-12V\""
-			(at 274.32 25.4 0)
-			(effects
-				(font
+			(at 278.13 20.32 0)
+			(effects
+				(font

Commit message: Reverse engineering progress
Connections:
- net -12V is gone; now on net +12V: J1.7 (Pin_7)
- net ~{WR}: now reaches U3.10 (~{WR})
- net ~{RD}: now reaches U3.13 (~{RD})
- net SERIAL CLOCK: now reaches U3.20 (CLK)
- net ~{TxC}: now reaches U3.9 (~{TxC})

Commit message: Further reverse engineering progress
Connections:
- net +5V: now also U3.26 (V_{CC})
- net GND: now also U3.4 (GND)
- net RESET: now reaches U3.21 (RESET)
- net ~{RESIN} (КР580ГФ24) renamed ~{RESIN}
Other:
- company: (none) -> Brett Hallen
- title: (none) -> Rhythm Keyboard (Ритм Клав)

Commit message: Reverse engineering updates
Parts:
- added C2, C3: 1µF, symbol Device:C
- added R7: 51KΩ, symbol Device:R
- added R8: 100KΩ, symbol Device:R
Connections:
- net GND: now also R8.2
- net at J2.3: now also C2.2, C3.2, R8.1
- new net: C2.1, C3.1, R7.2
Other:
- moved on the sheet: J2

Commit message: 19-May reverse engineering progress
Connections:
- net GND: now also U3.17 (~{CTS})
- net ~{TxC}: now also U3.25 (~{RxC})
- net A0: now reaches U3.12 (C/~{D})
- no-connect marks 2 -> 9
Changed lines of the file:
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@@
 	(generator "eeschema")
 	(generator_version "9.0")
-	(paper "A4")
+	(paper "A3")
 	(title_block
 		(title "Rhythm Keyboard (Ритм Клав)")
@@
 	)
 	(no_connect
+		(at 107.95 104.14)
+	)
+	(no_connect
+		(at 107.95 83.82)
+	)
+	(no_connect
+		(at 107.95 81.28)
+	)
+	(no_connect
+		(at 107.95 101.6)
+	)
+	(no_connect
+		(at 107.95 86.36)
+	)
+	(no_connect
+		(at 82.55 104.14)
+	)
+	(no_connect
 		(at 111.76 160.02)
 	)
@@
 		(at 96.52 160.02)
 	)
+	(no_connect
+		(at 107.95 96.52)
+	)
 	(wire
 		(pts
@@
 		)
 	)
+	(global_label "A0"
+		(shape input)
+		(at 82.55 99.06 180)
+		(fields_autoplaced yes)
+		(effects
+			(font
+				(size 1.27 1.27)
+			)
+			(justify right)
+		)
+		(property "Intersheetrefs" "${INTERSHEET_REFS}"
+			(at 77.2667 99.06 0)
+			(effects
+				(font
+					(size 1.27 1.27)
+				)
+				(justify right)
+				(hide yes)
+			)
+		)
+	)
 	(global_label "D3"
 		(shape input)
@@
 		)
 	)
+	(global_label "~{TxC}"
+		(shape input)
+		(at 107.95 78.74 0)
+		(fields_autoplaced yes)
+		(effects
+			(font
+				(size 1.27 1.27)
+			)
+			(justify left)
+		)
+		(property "Intersheetrefs" "${INTERSHEET_REFS}"
+			(at 114.2009 78.74 0)
+			(effects
+				(font
+					(size 1.27 1.27)
+				)
+				(justify left)
+				(hide yes)
+			)
+		)
+	)
 	(global_label "+12V"
 		(shape input)
@@
 				(hide yes)
 			)
+		)
+	)
+	(global_label "GND"
+		(shape input)
+		(at 107.95 99.06 0)
+		(fields_autoplaced yes)
+		(effects
+			(font
+				(size 1.27 1.27)
+			)
+			(justify left)
+		)
+		(property "Intersheetrefs" "${INTERSHEET_REFS}"
+			(at 114.8057 99.06 0)
+			(effects
+				(font
+					(size 1.27 1.27)
+				)
+				(justify left)
+				(hide yes)
+			)
