File: Schematic_Scraps/Keyboard.kicad_sch (KiCad schematic)
At the start: 1 part, among them U16 КР580ВВ55А/8255

Commit message: 19-May reverse engineering progress
Parts:
- added D2, D3, D4, D5, D6, D7, D8, D9: D, symbol Device:D
- added SW1: F1, symbol Switch:SW_Push_45deg
- added SW10: 5, symbol Switch:SW_Push_45deg
- added SW11: 6, symbol Switch:SW_Push_45deg
- added SW12: 7, symbol Switch:SW_Push_45deg
- added SW13: 8, symbol Switch:SW_Push_45deg
- added SW14: 9, symbol Switch:SW_Push_45deg
- added SW15: 0, symbol Switch:SW_Push_45deg
- added SW16: -, symbol Switch:SW_Push_45deg
- added SW17: =, symbol Switch:SW_Push_45deg
- added SW18: DEL, symbol Switch:SW_Push_45deg
- added SW19: RESET?, symbol Switch:SW_Push_45deg
- added SW2: F2, symbol Switch:SW_Push_45deg
- added SW20: Q, symbol Switch:SW_Push_45deg
- added SW21: W, symbol Switch:SW_Push_45deg
- added SW22: E, symbol Switch:SW_Push_45deg
- added SW23: R, symbol Switch:SW_Push_45deg
- added SW24: T, symbol Switch:SW_Push_45deg
- added SW25: Y, symbol Switch:SW_Push_45deg
- added SW26: U, symbol Switch:SW_Push_45deg
- added SW27: I, symbol Switch:SW_Push_45deg
- added SW28: O, symbol Switch:SW_Push_45deg
- added SW29: P, symbol Switch:SW_Push_45deg
- added SW3: F3, symbol Switch:SW_Push_45deg
- added SW30: [, symbol Switch:SW_Push_45deg
- added SW31: ], symbol Switch:SW_Push_45deg
- added SW32: \, symbol Switch:SW_Push_45deg
- added SW33: CAPS LOCK, symbol Switch:SW_Push_45deg
- added SW34: A, symbol Switch:SW_Push_45deg
- added SW35: S, symbol Switch:SW_Push_45deg
- added SW36: D, symbol Switch:SW_Push_45deg
- added SW37: F, symbol Switch:SW_Push_45deg
- added SW38: G, symbol Switch:SW_Push_45deg
- added SW39: H, symbol Switch:SW_Push_45deg
- added SW4: F4, symbol Switch:SW_Push_45deg
- added SW40: J, symbol Switch:SW_Push_45deg
- added SW41: K, symbol Switch:SW_Push_45deg
- added SW42: L, symbol Switch:SW_Push_45deg
- added SW43: ;, symbol Switch:SW_Push_45deg
- added SW44: ', symbol Switch:SW_Push_45deg
- added SW45: ENTER, symbol Switch:SW_Push_45deg
- added SW46: CTRL, symbol Switch:SW_Push_45deg
- added SW47: Z, symbol Switch:SW_Push_45deg
- added SW48: X, symbol Switch:SW_Push_45deg
- added SW49: C, symbol Switch:SW_Push_45deg
- added SW5: `, symbol Switch:SW_Push_45deg
- added SW50: V, symbol Switch:SW_Push_45deg
- added SW51: B, symbol Switch:SW_Push_45deg
- added SW52: N, symbol Switch:SW_Push_45deg
- added SW53: M, symbol Switch:SW_Push_45deg
- added SW54: ,, symbol Switch:SW_Push_45deg
- added SW55: ., symbol Switch:SW_Push_45deg
- added SW56: /, symbol Switch:SW_Push_45deg
- added SW57: РУС ЛАТ, symbol Switch:SW_Push_45deg
- added SW58: ALT, symbol Switch:SW_Push_45deg
- added SW59: <--, symbol Switch:SW_Push_45deg
- added SW6: 1, symbol Switch:SW_Push_45deg
- added SW60: -->, symbol Switch:SW_Push_45deg
- added SW61: SPACE1, symbol Switch:SW_Push_45deg
- added SW62: SPACE2, symbol Switch:SW_Push_45deg
- added SW7: 2, symbol Switch:SW_Push_45deg
- added SW8: 3, symbol Switch:SW_Push_45deg
- added SW9: 4, symbol Switch:SW_Push_45deg
Connections:
- net at U16.12 (PC5): now also D2.1 (K)
- net at U16.18 (PB0): now also D8.1 (K)
- net at U16.19 (PB1): now also D9.1 (K)
- net at U16.22 (PB4): now also D7.1 (K)
- net at U16.23 (PB5): now also D4.1 (K)
- net at U16.24 (PB6): now also D6.1 (K)
- net at U16.25 (PB7): now also D3.1 (K)
- net at U16.39 (PA5): now also D5.1 (K)
- new net: SW20.2, SW21.2, SW22.2, SW26.2
- new net: SW1.2, SW10.2, SW11.2, SW5.2, SW7.2
- new net: SW13.2, SW14.2, SW17.2
- new net: SW25.1, SW32.1, SW43.1, SW53.1, SW60.1, SW9.1
- new net: SW12.1, SW18.1, SW27.1, SW40.1, SW41.1, SW45.1, SW52.1
- new net: SW55.2, SW56.2
- new net: SW28.2, SW29.2, SW30.2, SW31.2
- new net: SW2.2, SW3.2
- new net: SW33.2, SW34.2, SW35.2, SW38.2, SW39.2
- new net: SW46.2, SW58.2
- new net: SW50.2, SW51.2, SW54.2
