File: Schematic/Interface.kicad_sch (KiCad schematic)
At the start: 13 parts, among them J1 Conn_01x09, J2 Cassette, U1 АОТ101АС (ILD74), U2 К555ТЛ2 (74LS14), U3 КР580ВВ51А (8251)

Commit message: Turning into a real schematic ...
Parts:
- added J4: СНП58-64, symbol Connector:DIN41612_02x32_AB
Connections:
- new net RDYIN: J4.a21 (Pin_a21)
- new net ~{STSTB}: J4.a27 (Pin_a27)
Changed lines of the file:
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@@
+		)
+	)
+	(global_label "RDYIN"
+		(shape input)
+		(at 196.85 207.01 180)
+		(fields_autoplaced yes)
+		(effects
+			(font
+				(size 1.27 1.27)
+			)
+			(justify right)
+		)
+		(property "Intersheetrefs" "${INTERSHEET_REFS}"
+			(at 188.3009 207.01 0)
+			(effects
+				(font
+					(size 1.27 1.27)
+				)
+				(justify right)
+				(hide yes)
+			)
 		)
 	)
@@
 		(property "Intersheetrefs" "${INTERSHEET_REFS}"
 			(at 75.6943 78.74 0)
+			(effects
+				(font
+					(size 1.27 1.27)
+				)
+				(justify right)
+				(hide yes)
+			)
+		)
+	)
+	(global_label "~{STSTB}"
+		(shape input)
+		(at 196.85 222.25 180)
+		(fields_autoplaced yes)
+		(effects
+			(font
+				(size 1.27 1.27)
+			)
+			(justify right)
+		)
+		(property "Intersheetrefs" "${INTERSHEET_REFS}"
+			(at 188.2406 222.25 0)
 			(effects
 				(font
@@
 					(unit 1)
 				)
+			)
+		)
+	)
+	(symbol
+		(lib_id "Connector:DIN41612_02x32_AB")
+		(at 201.93 194.31 0)
+		(unit 1)
+		(exclude_from_sim no)
+		(in_bom yes)
+		(on_board yes)
+		(dnp no)
+		(fields_autoplaced yes)
+		(property "Reference" "J4"
+			(at 203.2 149.86 0)
+			(effects
+				(font
+					(size 1.27 1.27)
+				)
+			)
+		)
+		(property "Value" "СНП58-64"
+			(at 203.2 152.4 0)
+			(effects
+				(font
+					(size 1.27 1.27)
+				)
+			)
+		)
+		(property "Footprint" ""
+			(at 201.93 194.31 0)
+			(effects
+				(font
+					(size 1.27 1.27)
+				)
+				(hide yes)
+			)
+		)
+		(property "Datasheet" "~"
+			(at 201.93 194.31 0)
+			(effects
+				(font
+					(size 1.27 1.27)
+				)
+				(hide yes)
+			)
+		)
+		(property "Description" "DIN41612 connector, double row (AB), 02x32, script generated (kicad-library-utils/schlib/autogen/connector/)"
+			(at 201.93 194.31 0)
+			(effects
+				(font
+					(size 1.27 1.27)
+				)
+				(hide yes)
+			)
+		)
+		(pin "a3"
+		)
+		(pin "a1"
+		)
+		(pin "a2"
+		)
+		(pin "a20"
+		)
+		(pin "a17"
+		)
+		(pin "a18"
+		)
+		(pin "a19"
+		)
+		(pin "a22"
+		)
+		(pin "a23"
+		)
+		(pin "a21"
+		)
+		(pin "a15"
+		)
+		(pin "a12"
+		)
+		(pin "a13"
+		)
+		(pin "a8"
+		)
+		(pin "a4"
+		)
+		(pin "a11"
+		)
+		(pin "a10"
+		)
+		(pin "a6"
+		)
+		(pin "a5"
+		)
+		(pin "a7"
+		)
+		(pin "a14"
+		)
+		(pin "a16"
+		)
+		(pin "a9"
+		)
+		(pin "b12"
+		)
+		(pin "b32"
+		)
+		(pin "b31"
+		)
+		(pin "b30"
+		)
+		(pin "b29"
+		)
+		(pin "b28"
+		)
+		(pin "b27"
+		)
+		(pin "b26"
+		)
+		(pin "b25"
+		)
+		(pin "b24"
+		)
+		(pin "b23"
+		)
+		(pin "b22"
+		)
+		(pin "b21"
+		)
+		(pin "b20"
+		)
+		(pin "b19"
+		)
+		(pin "b18"
+		)
+		(pin "b17"
+		)
+		(pin "b16"
+		)
+		(pin "b15"
+		)
+		(pin "b14"
+		)
+		(pin "b13"
+		)
+		(pin "a27"
+		)
+		(pin "b8"
+		)
+		(pin "b2"
+		)
+		(pin "a28"
+		)
+		(pin "a29"
+		)
+		(pin "a30"
+		)
+		(pin "a31"
+		)
+		(pin "a32"
+		)
+		(pin "b1"
+		)
+		(pin "a24"
+		)
+		(pin "b5"
+		)
+		(pin "b4"
+		)
+		(pin "b7"
+		)
+		(pin "b6"
+		)
+		(pin "b3"
+		)
+		(pin "b11"
+		)
+		(pin "a25"
+		)
+		(pin "a26"
+		)
+		(pin "b9"
+		)
+		(pin "b10"
+		)
+		(instances
+			(project "Schematic_Scraps"
+				(path "/194ce53b-cb13-451b-b32c-a7ec2b2ef170/2339c77a-ee2e-45eb-9203-d71b39a195c4"
+					(reference "J4")
+					(unit 1)
+				)
